Commit message: feat: 新增URDF模型点云采样功能 fix: 修改默认值和格式错误 style: 代码格式化调整

File: assets/screwdriver/screwdriver_limit_no_inertial.urdf (robot description, URDF)
Before this commit: robot screwdriver_on_the_table, 7 links, 6 joints
Joints:
- joint screwdriver_body_cap_joint: limit (none) -> lower=-1.57 upper=1.57 effort=10 velocity=0.5
- joint screwdriver_body_marker_joint: limit (none) -> lower=-1.57 upper=1.57 effort=10 velocity=0.5
- joint screwdriver_stick_body_joint: limit (none) -> lower=-1.57 upper=1.57 effort=10 velocity=0.5
- joint table_screwdriver_joint_3: limit (none) -> lower=-1.57 upper=1.57 effort=10 velocity=0.5
